File: Blinds_Stepper - Nano/Blinds_Stepper.sch (EAGLE design)
At the start: 22 parts

Commit message: clean up Blinds Stepper
Parts:
- added D1: (no value), wirepad:1,6/0,8
Connections:
- new net D13: D1.P, U$2.D13
Changed lines of the file:
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@@
 <part name="A6" library="wirepad" deviceset="1,6/0,8" device=""/>
 <part name="A7" library="wirepad" deviceset="1,6/0,8" device=""/>
+<part name="D1" library="wirepad" deviceset="1,6/0,8" device=""/>
 </parts>
 <sheets>
@@
 <attribute name="VALUE" x="102.362" y="44.577" size="1.778" layer="96" rot="R90"/>
 </instance>
+<instance part="D1" gate="P" x="137.16" y="45.72" smashed="yes" rot="R180">
+<attribute name="VALUE" x="138.303" y="49.022" size="1.778" layer="96" rot="R180"/>
+</instance>
 </instances>
 <busses>
@@
 </segment>
 </net>
+<net name="D13" class="0">
+<segment>
+<pinref part="U$2" gate="G$1" pin="D13"/>
+<wire x1="114.3" y1="63.5" x2="119.38" y2="63.5" width="0.1524" layer="91"/>
+<label x="114.3" y="63.5" size="1.778" layer="95"/>
+</segment>
+<segment>
+<pinref part="D1" gate="P" pin="P"/>
+<wire x1="134.62" y1="45.72" x2="129.54" y2="45.72" width="0.1524" layer="91"/>
+<label x="129.54" y="45.72" size="1.778" layer="95"/>
+</segment>
+</net>
