File: Nano Breakout/Nano Breakout.brd (EAGLE design)
At the start: 45.4 x 49.5 mm, 7 parts

Commit message: remove old dead projects, add esp-01 sensor stuff
Parts:
- added SJ1, SJ2, SJ3, SJ4: JUMPER-PAD-3-NOFULL_BOX_SILK, SparkFun-Passives:PAD-JUMPER-3-NO_YES_SILK_FULL_BOX
- moved U$1 3.59 mm to (24.1, 24.1)
- moved JP3 3.59 mm to (6.35, 25.4)
- moved JP1 3.59 mm to (8.89, 25.4)
- moved JP2 3.59 mm to (3.81, 25.4)
- moved JP4 3.59 mm to (31.8, 25.4)
- moved JP5 3.59 mm to (34.3, 25.4)
- moved JP6 3.59 mm to (36.8, 25.4)
Connections:
- removed net 5V: JP2.1, JP2.10, JP2.11, JP2.12, JP2.13, JP2.14, JP2.15, JP2.2, JP2.3, JP2.4, JP2.5, JP2.6, JP2.7, JP2.8, JP2.9, JP4.4, JP6.1, JP6.10, JP6.11, JP6.12, JP6.13, JP6.14, JP6.15, JP6.2, JP6.3, JP6.4, JP6.5, JP6.6, JP6.7, JP6.8, JP6.9, U$1.5V
- new net N$1: JP4.4, SJ1.3, SJ2.1, SJ3.1, SJ4.3, U$1.5V
- new net N$17: JP4.14, SJ1.1, SJ2.3, SJ3.3, SJ4.1, U$1.3V3
- new net N$2: JP2.10, JP2.11, JP2.12, JP2.13, JP2.14, JP2.15, JP2.8, JP2.9, SJ3.2
- new net PLB: JP2.1, JP2.2, JP2.3, JP2.4, JP2.5, JP2.6, JP2.7, SJ1.2
- new net PRB: JP6.10, JP6.11, JP6.12, JP6.13, JP6.14, JP6.15, JP6.9, SJ2.2
- net N$4: now also JP6.1, JP6.2, JP6.3, JP6.4, JP6.5, JP6.6, JP6.7, JP6.8, SJ4.2; no longer JP4.14, U$1.3V3
Routing:
- net 5V: track 137.8 -> 0.00 mm
- net N$17: track 0.00 -> 70.7 mm, vias 0 -> 4
- net N$1: track 0.00 -> 69.8 mm
- net N$2: track 0.00 -> 32.3 mm
- net PRB: track 0.00 -> 31.0 mm
- net PLB: track 0.00 -> 29.7 mm
- net N$4: track 3.81 -> 32.3 mm
Other:
- board size 45.4 x 49.5 mm -> 40.6 x 49.8 mm
